File: FinalProject/misc/DocImg/WalleBoard/walle.brd (EAGLE design)
At the start: 37.8 x 21.8 mm, 6 parts, among them U1 Tiny45-20-SMT

Commit message: finalproject
Parts:
- removed U$1: ULTRASONIC-HC-SR04, diy-modules:ULTRASONIC-HC-SR04
- added JP1: (no value), jumper:JP4
- moved C1 6.03 mm to (26.7, 13.6)
- moved R1 3.98 mm to (26.4, 5.84), turned to 0 degrees
- moved U$2 1.14 mm to (7.62, 6.48)
Connections:
- net ECHO: now also JP1.3; no longer U$1.3
- net GND: now also JP1.4; no longer U$1.4
- net N$1: now also JP1.1; no longer U$1.1
- net TRIG: now also JP1.2; no longer U$1.2
Routing:
- net GND: track 30.5 -> 19.1 mm
- net MOSI: track 18.7 -> 12.3 mm
- net N$3: track 11.7 -> 6.60 mm
- net PB5: track 15.1 -> 20.2 mm
- net SCK: track 32.8 -> 29.8 mm
- net ECHO: track 7.04 -> 9.86 mm
- net TRIG: track 6.78 -> 8.81 mm
- net N$1: track 64.4 -> 63.3 mm
- added copper zone on layer 1, net N$2
Other:
- board size 37.8 x 21.8 mm -> 37.8 x 24.9 mm
- board text removed: "00Final"
