File: FinalProject/misc/DocImg/WalleBoard/walle.sch (EAGLE design)
At the start: 6 parts, among them U1 Tiny45-20-SMT

Commit message: finalproject
Parts:
- removed U$1: ULTRASONIC-HC-SR04, diy-modules:ULTRASONIC-HC-SR04
- added JP1: (no value), jumper:JP4E
Connections:
- net ECHO: now also JP1.3; no longer U$1.ECHO
- net GND: now also JP1.4; no longer U$1.GND
- net N$1: now also JP1.1; no longer U$1.VCC
- net TRIG: now also JP1.2; no longer U$1.TRIG
Changed lines of the file:
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@@
 </classes>
 <parts>
-<part name="U$1" library="diy-modules" deviceset="ULTRASONIC-HC-SR04" device=""/>
 <part name="U$2" library="fab" deviceset="AVRISP" device="SMD"/>
 <part name="C1" library="fab" deviceset="CAP-UNPOLARIZED" device=""/>
@@
 <part name="U1" library="SparkFun-DigitalIC" deviceset="ATTINY45" device="TINY45-20-SMT" value="Tiny45-20-SMT"/>
 <part name="GND2" library="supply1" deviceset="GND" device=""/>
+<part name="JP1" library="jumper" deviceset="JP4E" device=""/>
 </parts>
 <sheets>
@@
 </plain>
 <instances>
-<instance part="U$1" gate="G$1" x="124.46" y="170.18"/>
 <instance part="U$2" gate="G$1" x="99.06" y="137.16"/>
 <instance part="C1" gate="&gt;NAME" x="154.94" y="139.7"/>
@@
 <instance part="U1" gate="G$1" x="139.7" y="106.68"/>
 <instance part="GND2" gate="1" x="116.84" y="99.06"/>
+<instance part="JP1" gate="G$1" x="124.46" y="157.48"/>
 </instances>
 <busses>
@@
 </segment>
 <segment>
-<pinref part="U$1" gate="G$1" pin="GND"/>
 <pinref part="GND1" gate="1" pin="GND"/>
 <wire x1="129.54" y1="154.94" x2="139.7" y2="154.94" width="0.1524" layer="91"/>
+<pinref part="JP1" gate="G$1" pin="4"/>
 </segment>
 <segment>
@@
 <net name="ECHO" class="0">
 <segment>
-<pinref part="U$1" gate="G$1" pin="ECHO"/>
 <wire x1="127" y1="154.94" x2="127" y2="147.32" width="0.1524" layer="91"/>
 <label x="127" y="149.86" size="1.778" layer="95"/>
+<pinref part="JP1" gate="G$1" pin="3"/>
 </segment>
 <segment>
@@
 <net name="TRIG" class="0">
 <segment>
-<pinref part="U$1" gate="G$1" pin="TRIG"/>
 <wire x1="124.46" y1="154.94" x2="124.46" y2="147.32" width="0.1524" layer="91"/>
 <label x="124.46" y="147.32" size="1.778" layer="95"/>
+<pinref part="JP1" gate="G$1" pin="2"/>
 </segment>
 <segment>
@@
 <pinref part="C1" gate="&gt;NAME" pin="1"/>
 <wire x1="142.24" y1="139.7" x2="144.78" y2="139.7" width="0.1524" layer="91"/>
-<pinref part="U$1" gate="G$1" pin="VCC"/>
 <wire x1="144.78" y1="139.7" x2="147.32" y2="139.7" width="0.1524" layer="91"/>
 <wire x1="147.32" y1="139.7" x2="149.86" y2="139.7" width="0.1524" layer="91"/>
@@
 <wire x1="154.94" y1="137.16" x2="154.94" y2="132.08" width="0.1524" layer="91"/>
 <wire x1="154.94" y1="132.08" x2="144.78" y2="132.08" width="0.1524" layer="91"/>
+<pinref part="JP1" gate="G$1" pin="1"/>
 </segment>
 </net>
