File: Week15/misc/week15files/networking-node.brd (EAGLE design)
At the start: 34 x 21.6 mm, 7 parts, among them J1ISP AVRISPSMD, J3BUS PINHD-2X2-SMD

Commit message: week11/13/15/final
Connections:
- removed net N$2: J1ISP.2, J3BUS.3
- net VCC: now also J1ISP.2, J3BUS.3, R1.1
Routing:
- net N$2: track 25.8 -> 0.00 mm
- net VCC: track 37.0 -> 45.1 mm
- net TX: track 32.0 -> 33.3 mm
- net MISO: track 10.8 -> 9.66 mm
- net SCK: track 10.8 -> 11.7 mm
- net RX: track 40.9 -> 41.4 mm
Other:
- board size 34 x 21.6 mm -> 36.2 x 25.1 mm
- board text added: "NODE"
